Commit message: change urdf to reflect correct rotation

File: src/robots/franka_robotiq_description/robots/panda_robotiq.urdf.xacro (robot description, xacro)
@@ -3,5 +3,5 @@
   <link name="panda_link8"/>
   <joint name="panda_robotiq_attachment_joint" type="fixed">
-    <origin xyz="0 0 0" rpy="0 0 ${pi/2}"/>
+    <origin xyz="0 0 0" rpy="0 0 ${pi/4}"/>
     <parent link="panda_link8"/>
     <child link="robotiq_arg2f_base_link"/>

Commit message: fix panda_robotiq rotation

File: src/robots/franka_robotiq_description/robots/panda_robotiq.urdf.xacro (robot description, xacro)
@@ -3,5 +3,5 @@
   <link name="panda_link8"/>
   <joint name="panda_robotiq_attachment_joint" type="fixed">
-    <origin xyz="0 0 0" rpy="0 0 ${pi/4}"/>
+    <origin xyz="0 0 0" rpy="0 0 ${pi/2}"/>
     <parent link="panda_link8"/>
     <child link="robotiq_arg2f_base_link"/>
